Commit message: fixing small issue

File: src/testbed_navigation/urdf/testbed.xacro (robot description, xacro)
@@ -1,7 +1,7 @@
 <?xml version="1.0" ?>
 <robot name="testbed" xmlns:xacro="http://www.ros.org/wiki/xacro">
-<xacro:include filename="$(find testbed_description)/urdf/materials.xacro" />
-<xacro:include filename="$(find testbed_description)/urdf/testbed.trans" />
-<xacro:include filename="$(find testbed_description)/urdf/testbed.gazebo" />
+<xacro:include filename="$(find testbed_navigation)/urdf/materials.xacro" />
+<xacro:include filename="$(find testbed_navigation)/urdf/testbed.trans" />
+<xacro:include filename="$(find testbed_navigation)/urdf/testbed.gazebo" />
 <link name="base_footprint">
   <visual>
@@ -21,5 +21,5 @@
     <origin xyz="0 0 0" rpy="0 0 0"/>
     <geometry>
-      <mesh filename="file://$(find testbed_description)/meshes/base_link.stl" scale="0.001 0.001 0.001"/>
+      <mesh filename="file://$(find testbed_navigation)/meshes/base_link.stl" scale="0.001 0.001 0.001"/>
     </geometry>
     <material name="silver"/>
@@ -28,5 +28,5 @@
     <origin xyz="0 0 0" rpy="0 0 0"/>
     <geometry>
-      <mesh filename="file://$(find testbed_description)/meshes/base_link.stl" scale="0.001 0.001 0.001"/>
+      <mesh filename="file://$(find testbed_navigation)/meshes/base_link.stl" scale="0.001 0.001 0.001"/>
     </geometry>
   </collision>
@@ -41,5 +41,5 @@
     <origin xyz="0.050476 -0.135241 -0.050004" rpy="0 0 0"/>
     <geometry>
-      <mesh filename="file://$(find testbed_description)/meshes/left_wheel_1.stl" scale="0.001 0.001 0.001"/>
+      <mesh filename="file://$(find testbed_navigation)/meshes/left_wheel_1.stl" scale="0.001 0.001 0.001"/>
     </geometry>
     <material name="silver"/>
@@ -48,5 +48,5 @@
     <origin xyz="0.050476 -0.135241 -0.050004" rpy="0 0 0"/>
     <geometry>
-      <mesh filename="file://$(find testbed_description)/meshes/left_wheel_1.stl" scale="0.001 0.001 0.001"/>
+      <mesh filename="file://$(find testbed_navigation)/meshes/left_wheel_1.stl" scale="0.001 0.001 0.001"/>
     </geometry>
   </collision>
@@ -61,5 +61,5 @@
     <origin xyz="0.175703 -0.108591 -0.084004" rpy="0 0 0"/>
     <geometry>
-      <mesh filename="file://$(find testbed_description)/meshes/caster_1.stl" scale="0.001 0.001 0.001"/>
+      <mesh filename="file://$(find testbed_navigation)/meshes/caster_1.stl" scale="0.001 0.001 0.001"/>
     </geometry>
     <material name="silver"/>
@@ -68,5 +68,5 @@
     <origin xyz="0.175703 -0.108591 -0.084004" rpy="0 0 0"/>
     <geometry>
-      <mesh filename="file://$(find testbed_description)/meshes/caster_1.stl" scale="0.001 0.001 0.001"/>
+      <mesh filename="file://$(find testbed_navigation)/meshes/caster_1.stl" scale="0.001 0.001 0.001"/>
     </geometry>
   </collision>
@@ -81,5 +81,5 @@
     <origin xyz="0.175703 0.184109 -0.084004" rpy="0 0 0"/>
     <geometry>
-      <mesh filename="file://$(find testbed_description)/meshes/caster_2.stl" scale="0.001 0.001 0.001"/>
+      <mesh filename="file://$(find testbed_navigation)/meshes/caster_2.stl" scale="0.001 0.001 0.001"/>
     </geometry>
     <material name="silver"/>
@@ -88,5 +88,5 @@
     <origin xyz="0.175703 0.184109 -0.084004" rpy="0 0 0"/>
     <geometry>
-      <mesh filename="file://$(find testbed_description)/meshes/caster_2.stl" scale="0.001 0.001 0.001"/>
+      <mesh filename="file://$(find testbed_navigation)/meshes/caster_2.stl" scale="0.001 0.001 0.001"/>
     </geometry>
   </collision>
@@ -101,5 +101,5 @@
     <origin xyz="-0.074297 -0.108591 -0.084004" rpy="0 0 0"/>
     <geometry>
-      <mesh filename="file://$(find testbed_description)/meshes/caster_3.stl" scale="0.001 0.001 0.001"/>
+      <mesh filename="file://$(find testbed_navigation)/meshes/caster_3.stl" scale="0.001 0.001 0.001"/>
     </geometry>
     <material name="silver"/>
@@ -108,5 +108,5 @@
     <origin xyz="-0.074297 -0.108591 -0.084004" rpy="0 0 0"/>
     <geometry>
-      <mesh filename="file://$(find testbed_description)/meshes/caster_3.stl" scale="0.001 0.001 0.001"/>
+      <mesh filename="file://$(find testbed_navigation)/meshes/caster_3.stl" scale="0.001 0.001 0.001"/>
     </geometry>
   </collision>
@@ -121,5 +121,5 @@
     <origin xyz="-0.074297 0.184109 -0.084004" rpy="0 0 0"/>
     <geometry>
-      <mesh filename="file://$(find testbed_description)/meshes/caster_4.stl" scale="0.001 0.001 0.001"/>
+      <mesh filename="file://$(find testbed_navigation)/meshes/caster_4.stl" scale="0.001 0.001 0.001"/>
     </geometry>
     <material name="silver"/>
@@ -128,5 +128,5 @@
     <origin xyz="-0.074297 0.184109 -0.084004" rpy="0 0 0"/>
     <geometry>
-      <mesh filename="file://$(find testbed_description)/meshes/caster_4.stl" scale="0.001 0.001 0.001"/>
+      <mesh filename="file://$(find testbed_navigation)/meshes/caster_4.stl" scale="0.001 0.001 0.001"/>
     </geometry>
   </collision>
@@ -141,5 +141,5 @@
     <origin xyz="0.04 0.033 -0.226509" rpy="0 0 0"/>
     <geometry>
-      <mesh filename="file://$(find testbed_description)/meshes/lidar_link_1.stl" scale="0.001 0.001 0.001"/>
+      <mesh filename="file://$(find testbed_navigation)/meshes/lidar_link_1.stl" scale="0.001 0.001 0.001"/>
     </geometry>
     <material name="silver"/>
@@ -148,5 +148,5 @@
     <origin xyz="0.04 0.033 -0.226509" rpy="0 0 0"/>
     <geometry>
-      <mesh filename="file://$(find testbed_description)/meshes/lidar_link_1.stl" scale="0.001 0.001 0.001"/>
+      <mesh filename="file://$(find testbed_navigation)/meshes/lidar_link_1.stl" scale="0.001 0.001 0.001"/>
     </geometry>
   </collision>
@@ -161,5 +161,5 @@
     <origin xyz="0.1 -0.05 -0.1612" rpy="0 0 0"/>
     <geometry>
-      <mesh filename="file://$(find testbed_description)/meshes/imu_link_1.stl" scale="0.001 0.001 0.001"/>
+      <mesh filename="file://$(find testbed_navigation)/meshes/imu_link_1.stl" scale="0.001 0.001 0.001"/>
     </geometry>
     <material name="silver"/>
@@ -168,5 +168,5 @@
     <origin xyz="0.1 -0.05 -0.1612" rpy="0 0 0"/>
     <geometry>
-      <mesh filename="file://$(find testbed_description)/meshes/imu_link_1.stl" scale="0.001 0.001 0.001"/>
+      <mesh filename="file://$(find testbed_navigation)/meshes/imu_link_1.stl" scale="0.001 0.001 0.001"/>
     </geometry>
   </collision>
@@ -181,5 +181,5 @@
     <origin xyz="0.1 0.14 -0.1612" rpy="0 0 0"/>
     <geometry>
-      <mesh filename="file://$(find testbed_description)/meshes/dummy_link_1.stl" scale="0.001 0.001 0.001"/>
+      <mesh filename="file://$(find testbed_navigation)/meshes/dummy_link_1.stl" scale="0.001 0.001 0.001"/>
     </geometry>
     <material name="silver"/>
@@ -188,5 +188,5 @@
     <origin xyz="0.1 0.14 -0.1612" rpy="0 0 0"/>
     <geometry>
-      <mesh filename="file://$(find testbed_description)/meshes/dummy_link_1.stl" scale="0.001 0.001 0.001"/>
+      <mesh filename="file://$(find testbed_navigation)/meshes/dummy_link_1.stl" scale="0.001 0.001 0.001"/>
     </geometry>
   </collision>
@@ -201,5 +201,5 @@
     <origin xyz="0.050503 0.210759 -0.050004" rpy="0 0 0"/>
     <geometry>
-      <mesh filename="file://$(find testbed_description)/meshes/right_wheel_1.stl" scale="0.001 0.001 0.001"/>
+      <mesh filename="file://$(find testbed_navigation)/meshes/right_wheel_1.stl" scale="0.001 0.001 0.001"/>
     </geometry>
     <material name="silver"/>
@@ -208,5 +208,5 @@
     <origin xyz="0.050503 0.210759 -0.050004" rpy="0 0 0"/>
     <geometry>
-      <mesh filename="file://$(find testbed_description)/meshes/right_wheel_1.stl" scale="0.001 0.001 0.001"/>
+      <mesh filename="file://$(find testbed_navigation)/meshes/right_wheel_1.stl" scale="0.001 0.001 0.001"/>
     </geometry>
   </collision>
